File: build/pcb/claude-micro.kicad_sch (KiCad schematic)
At the start: 89 parts, among them SW1 Kailh Choc v1, SW10 Kailh Choc v1, SW11 Kailh Choc v1, SW12 Kailh Choc v1, SW13 Kailh Choc v1, SW2 Kailh Choc v1, SW3 Kailh Choc v1, SW4 Kailh Choc v1, SW5 Kailh Choc v1, SW6 Kailh Choc v1, SW7 Kailh Choc v1, SW8 Kailh Choc v1, SW9 Kailh Choc v1, U2 74LVC1G17

Commit message: Switch to clear MX switches; fix the EasyEDA project wrapper
Two changes.

EasyEDA
-------
The project wrapper now matches what EasyEDA 6.5 actually writes: docType is
the string "5" (not the integer 5), colors is an object, editorVersion sits at
the top level alongside a description, and each sheet carries its own string
docType and description. The 4.x shape I had reverse-engineered from an older
exported file would not round-trip. The structural test now asserts the exact
key set and types on both the project and the sheet.

Switches
--------
Kailh Choc low-profile replaced with clear-housing MX-compatible switches,
5-pin PCB mount. That is not a drop-in: MX needs a 19.05 mm grid where Choc
ran at 18 x 17, so the whole device re-derives from the config.

- footprint: two contacts at (-3.81, 2.54) and (2.54, 5.08), centre boss and
  two locating posts, 14 mm plate cutout, both contacts on the south half so
  the north half stays clear for the per-key LED in the switch's light window
- keycaps: 18 x 18 mm with a cross socket instead of Choc's twin posts, so
  bought MX caps drop in as an alternative to printing them
- Z stack rebuilt for 4 mm travel and an 11.6 mm body; the taller stack means
  the encoder now takes a stock 12.5 mm shaft rather than a trimmed one
- board 128 x 88 -> 159 x 102 mm, case 134 x 94 -> 165 x 108 mm, and the MCU
  module moved to the gutters of the new grid (pin columns at x=9.25 and
  x=27.03) so its through-holes still miss every top-side pad
- switches render translucent in the viewer to match the clear housings

The switch footprint name is now read from the config rather than hardcoded in
the ERC and two tests, which is what caught the 0-switches-for-13-keys error
after the swap.

Rebuilt and re-verified: 141/141 connections routed, 0 DRC errors, 0 warnings,
9/9 meshes watertight, 36/36 checks passing.

Co-Authored-By: Claude Opus 5 <noreply@anthropic.com>
Claude-Session: https://claude.ai/code/session_018r1gdNJN1A3uPDEU4991Ag
Parts:
- SW1, SW10, SW11, SW12, SW13, SW2, SW3, SW4, SW5, SW6, SW7, SW8, SW9: value Kailh Choc v1 -> MX clear; footprint claude-micro:Choc_v1 -> claude-micro:MX_PCB; symbol claude-micro:Choc_v1 -> claude-micro:MX_PCB
